File: dpowerV1.kicad_sch (KiCad schematic)
At the start: 67 parts, among them J1 USB_A, J2 USB_C_Receptacle_USB2.0_16P, Q1 8205S_C2762930, Q2 8205S_C2762930, Q3 AO4435, Q4 BSS138, Q6 AO4435, U1 DW01A_C2927799, U2 AP2112K-3.3TRG1(MS), U3 FP6296XR-G1, U4 IP2161, U5 SRV05-4, U6 SRV05-4, U7 CN3791, U8 CH224K

Commit message: update
Parts:
- removed D4: SK54C, Diode_SMD:D_SMC_Handsoldering, symbol lcsc:SK54C_C5449119
- added D1: SK54C_C5449119, Diode_SMD:D_SMC_Handsoldering, symbol lcsc:SK54C_C5449119
- added J3: Conn_01x05_Pin, symbol Connector:Conn_01x05_Pin
- added R21: R10k, Resistor_SMD:R_0508_1220Metric_Pad1.12x2.15mm_HandSolder, symbol Device:R
- added U9: PY32F002AW15S6TU, Package_SO:SOP-16_4.4x10.4mm_P1.27mm, symbol lcsc:PY32F002AW15S6TU
- BT1, BT2: footprint lcsc_footprints:C5290176_BAT-TH_BH-18650-A1AJ005 -> lcsc_footprints:C5290175_BAT-TH_BH-18650-A1AJ006; LCSC C5290176 -> C5290175
- R16: value R6k8 -> R24k
- R20: footprint Resistor_SMD:R_0508_1220Metric_Pad1.12x2.15mm_HandSolder -> Resistor_SMD:R_1206_3216Metric_Pad1.30x1.75mm_HandSolder
- U5: footprint Package_TO_SOT_SMD:SOT-23-6 -> Package_TO_SOT_SMD:SOT-23-6_Handsoldering
Connections:
- net +3V3: now also J3.4 (Pin_4), R21.2, U9.4 (VCC)
- net B+: no longer U2.3 (EN)
- net BOOST_LX: now also D2.2 (A), L1.2, U3.1 (LX), U3.2 (LX)
- net CHARG_DRAIN: now also D1.1 (C)
- net GND: now also D1.2 (A), J3.3 (Pin_3), U9.13 (VSS); no longer C2.2, U2.2 (GND)
- new net: C2.2, U2.2 (GND)
- new net LDO_EN: U2.3 (EN)
- new net PY32_RESET: J3.5 (Pin_5), R21.1, U9.8 (PF2-NRST)
- new net PY32_SWC: J3.1 (Pin_1), U9.7 (PA14-SWC)
- new net PY32_SWD: J3.2 (Pin_2), U9.6 (PA13-SWD)

Commit message: update
Parts:
- added C28, C29: C100nF, Capacitor_SMD:C_0805_2012Metric_Pad1.18x1.45mm_HandSolder, symbol Device:C
- added C30: C10uF, Capacitor_SMD:C_0805_2012Metric_Pad1.18x1.45mm_HandSolder, symbol Device:C
- added C31, C32, C33: C0.1uF, Capacitor_SMD:C_0805_2012Metric_Pad1.18x1.45mm_HandSolder, symbol Device:C
- added D4: BAT54C, Package_TO_SOT_SMD:SOT-23, symbol Diode:BAT54C
- added D5, D6, D7, D8: LED, symbol Device:LED
- added D9: LED_GREEN, symbol Device:LED
- added JP1: SolderJumper_3_Open, Jumper:SolderJumper-3_P2.0mm_Open_TrianglePad1.0x1.5mm, symbol Jumper:SolderJumper_3_Open
- added Q5: AO4435, danad_footprints:SOIC-8_3.9x4.9mm_P1.27mm_AO4435_HandSolder, symbol Transistor_FET:AO3401A
- added R22, R34: R24k, Resistor_SMD:R_0508_1220Metric_Pad1.12x2.15mm_HandSolder, symbol Device:R
- added R23: R26k, Resistor_SMD:R_0508_1220Metric_Pad1.12x2.15mm_HandSolder, symbol Device:R
- added R24, R25, R26, R27, R32: R100k, Resistor_SMD:R_0508_1220Metric_Pad1.12x2.15mm_HandSolder, symbol Device:R
- added R28, R29, R30, R31, R37: R470, Resistor_SMD:R_0508_1220Metric_Pad1.12x2.15mm_HandSolder, symbol Device:R
- added R33, R35: R10k, Resistor_SMD:R_0508_1220Metric_Pad1.12x2.15mm_HandSolder, symbol Device:R
- added R36: R2k, Resistor_SMD:R_0508_1220Metric_Pad1.12x2.15mm_HandSolder, symbol Device:R
- added SW1: SW_SPDT, lcsc_footprints:C431548_SW-TH_SK12D07VG5-1, symbol Switch:SW_SPDT
- added SW2: TC-6615-8.0, lcsc_footprints:C7528686_SW-TH_4P-L7_5-W8_0-P4_50, symbol lcsc:TC-6615-8_0
- D1: footprint Diode_SMD:D_SMA -> Diode_SMD:D_SMA_Handsoldering
- J2: footprint Connector_USB:USB_C_Receptacle_GCT_USB4105-xx-A_16P_TopMnt_Horizontal -> danad_footprints:USB_C_Receptacle_GCT_USB4105-xx-A_16P_TopMnt_Horizontal_HandSolder
- R17: value R10k -> R100k
- U9: footprint Package_SO:SOP-16_4.4x10.4mm_P1.27mm -> danad_footprints:SOP-16_4.4x10.4mm_P1.27mm_Handsolder
Connections:
- net +3V3: now also C29.2, D9.2 (A), JP1.2 (C), JP1.3 (B), R28.2, R29.2, R30.2, R31.2; no longer J3.4 (Pin_4)
- net B+: now also R25.2
- net BOOST_EN: now also U9.10 (PF1-OSCOUT), R27.1
- net GND: now also C2.2, U2.2 (GND), C28.1, C29.1, C30.2, C33.2, R22.2, R24.1, R26.2, R27.2, R33.2, R36.1, SW1.2 (B), SW2.1
- net LDO_EN: now also U9.9 (PF0-OSCIN), D4.2; no longer U2.3 (EN)
- net VBUS_GATE_PULLUP: now also C32.1
- net VBUS_IN: now also C30.1, Q5.2 (S), R23.1, R32.1; no longer C21.2, C22.2, C23.2, C26.2, C27.2, Q6.2 (S), R18.1, U7.9 (VCC)
- net ~CHRG: now also U9.11 (PA0)
- net BOOST_OUT: now reaches C11.1, C12.1, C13.1, C15.1, C16.1, D2.1 (C), Q3.2 (S), R17.2, R5.2, R8.2
- net BOOST_OUT: now also C32.2
- net at U7.6 (MPPT): now also R18.1, R34.2; no longer R18.2
- net at U9.1 (PA7): now also C28.2, R25.1, R26.1
- net at U9.12 (PA1): now also D5.1 (K)
- net at U9.14 (PA2): now also D6.1 (K)
- net at U9.15 (PA3): now also D7.1 (K)
- net at U9.16 (PA6): now also D8.1 (K)
- net PB0: now reaches U9.2 (PB0)
- net PB0: now also SW2.2
- net PB1: now reaches U9.3 (PB1)
- net PB1: now also SW1.1 (A)
- net ~DONE renamed ~CHARG_DONE
- net ~CHARG_DONE: now also R37.1
- new net: C31.2, C33.1, Q5.1 (G), R32.2, R33.1
- new net: D4.1, R22.1, R23.2
- new net: D9.1 (K), R37.2
- new net: D5.2 (A), R28.1
- new net: D8.2 (A), R31.1
- new net: D7.2 (A), R30.1
- new net: R34.1, R35.2
- new net: D6.2 (A), R29.1
- new net: D4.3, R24.2, U2.3 (EN)
- new net: R35.1, R36.2
- new net CHARG_VCC: C21.2, C22.2, C23.2, C26.2, C27.2, C31.1, Q5.3 (D), Q6.2 (S), R18.2, U7.9 (VCC)
- new net PY32_HEADER_4: J3.4 (Pin_4), JP1.1 (A)
- no-connect marks 13 -> 17
Other:
- moved on the sheet: C18, C19, C2, C20, C21, C22, C23, C24, C25, C26, C27, C3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

Commit message: update
Parts:
- C31: value C0.1uF -> C100nF
- C33: value C0.1uF -> C47nF
- R33: value R10k -> R100k
Connections:
- net CHARG_VCC: now also C33.1; no longer C31.1
- net GND: no longer C33.2
- net VBUS_IN: now also C31.1; no longer R32.1
- new net: C31.2, C33.2, Q5.1 (G), R32.1
- new net: R32.2, R33.1
